File: adapter/adapter.kicad_pcb (KiCad board)
At the start: 2 copper layers, 96 x 46 mm, 18 parts, among them J1 Conn_02x13_Top_Bottom, J10 Screw_Terminal_01x02, J11 Screw_Terminal_01x02, J12 Screw_Terminal_01x02, J13 Screw_Terminal_01x02, J14 Screw_Terminal_01x02, J2 Screw_Terminal_01x02, J3 Screw_Terminal_01x02, J4 Screw_Terminal_01x02, J5 Screw_Terminal_01x02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

Commit message: Finish routing
Routing:
- net /25: track 0.00 -> 23.9 mm
- net /26: track 0.00 -> 23.3 mm
- net /13: track 0.00 -> 23.3 mm
- net /12: track 0.00 -> 20.6 mm
- net /24: track 0.00 -> 19.6 mm
- net /11: track 0.00 -> 18.5 mm
- net /23: track 0.00 -> 17.9 mm
- net /10: track 0.00 -> 17.3 mm
- net /14: track 0.00 -> 17.1 mm
- net /1: track 0.00 -> 17.1 mm
- net /22: track 0.00 -> 16.4 mm
- net /2: track 0.00 -> 15.8 mm
- net /15: track 0.00 -> 15.8 mm
- net /9: track 0.00 -> 14.8 mm
- net /3: track 0.00 -> 14.8 mm
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- added copper zone on B.Cu, net (none)
Other:
- net class Default: clearance 0.2 -> 0.4
- rule trace_clearance: 0.2 -> 0.4
- board text added: "1"
- board text added: "1 2 3 4 5 6"
- board text added: "13 26"
- board text added: "25 24 23 22 21 20 19 18 17 16 15 14"
- board text added: "7 8 9 10 11 12"
- board text added: "IDC 2x13 to screw terminals adapter, Roman Pavelka 2021-09"

Commit message: Fix small mistakes
Routing:
- net /3: track 14.8 -> 13.3 mm
- net /1: track 17.1 -> 16.6 mm

Commit message: Checked if it still works in KiCAD 8 and updated
Other:
- net class Default removed
